Commit message: adapt functions for new angle measurements

File: ROS_MoveIt/multicar.urdf (robot description, URDF)
Before this commit: robot Multicar, 13 links, 12 joints
Joints:
- joint rot_dreharm_hauptarm: limit lower=3.4746 upper=5.3586 effort=1000.0 velocity=0.5 -> lower=3.6826 upper=4.9392 effort=1000.0 velocity=0.5
- joint rot_hauptarm_nebenarm: limit lower=3.5095 upper=5.82963 effort=1000.0 velocity=0.5 -> lower=3.5168 upper=5.7159 effort=1000.0 velocity=0.5
- joint rot_nebenarm_schnellwechselsystem: limit lower=1.60489 upper=4.553 effort=1000.0 velocity=0.5 -> lower=1.8064 upper=4.7647 effort=1000.0 velocity=0.5
